File: Hardware/PUTM_EV_Frontbox_2023/programator.kicad_sch (KiCad schematic)
At the start: 2 parts, among them U32 STLINK-V3MODS

Commit message: Free PB0-Boot pin
Parts:
- renumbered F6 to F5
Changed lines of the file:
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@@
   (symbol (lib_id "Device:Fuse_Small") (at 80.01 69.85 0) (unit 1)
     (in_bom yes) (on_board yes) (dnp no) (fields_autoplaced)
-    (property "Reference" "F6" (at 80.01 64.77 0)
+    (property "Reference" "F5" (at 80.01 64.77 0)
       (effects (font (size 1.27 1.27)))
     )
@@
       (project "PUTM_EV_Frontbox_2023"
         (path "/b652b05a-4e3d-4ad1-b032-18886abe7d45/dd0098ec-f4e0-48aa-9050-ddfd0a2e4304"
-          (reference "F6") (unit 1)
+          (reference "F5") (unit 1)
         )
       )

Commit message: Fixed production issues
Parts:
- F5: footprint Fuse:Fuse_1206_3216Metric_Pad1.42x1.75mm_HandSolder -> Fuse:Fuse_0805_2012Metric
