File: Hardware/PUTM_EV_Frontbox_2023/PUTM_EV_Frontbox_2023.kicad_pcb (KiCad board)
At the start: 4 copper layers, 97 x 70 mm, 275 parts, among them J1 Conn_02x16_Counter_Clockwise, K1 FINDER-32.21-x000, Q1 NX7002AK, U1 LM4040C33FTA, U10 MCP6001, U11 FODM217B, U12 TLP291-4, U13 TLP291-4, U14 MCP2542FDxMF, U15 MCP6002-xMC, U16 MCP6N11-005, U17 MCP6001, U18 MCP6002-xMC, U19 MCP6N11-005, U2 STM32G473RCTx, U20 MCP6001, U21 MCP6N11-005, U22 MCP6001, U23 MCP6N11-005, U24 MCP6001, U25 MCP6N11-005, U26 MCP6001, U27 MCP6N11-005, U28 MCP6001, U29 MCP6N11-005, U3 IMS330DHCX, U30 MCP6001, U31 STLINK-V3MODS, U4 TLV743P, U5 LM62440-Q1, U6 TLV743P, U7 TLV743P, U8 MCP2542FDxMF, U9 MCP6N11-005, Y1 ABM8G-48.000MHZ

Commit message: Free PB0-Boot pin
Parts:
- added F5: Fuse_Small, Fuse:Fuse_1206_3216Metric_Pad1.42x1.75mm_HandSolder, F.Cu at (2.48, 1.15)
- added R101: 10k, Resistor_SMD:R_0603_1608Metric, B.Cu at (203.0, 95.4)
- added R102: 10k, Resistor_SMD:R_0603_1608Metric, B.Cu at (203.0, 97.0)
- renumbered U31 to U32
Connections:
- U2 pad 58: unconnected-(U2-PB5-Pad58) -> /Sense_Right_Wheel
- U2 pad 59: /Sense_Right_Wheel -> /Sense_overtravel
- U2 pad 60: /Sense_overtravel -> /Sense_right
- U2 pad 61: /Sense_right -> Net-(U2-PB8)
Routing:
- net Net-(U2-PB8): track 0.00 -> 7.11 mm, vias 0 -> 1
- net +3.3V: track 224.5 -> 231.1 mm
- net GND: track 265.9 -> 267.5 mm, vias 157 -> 158

Commit message: Fixed production issues
Parts:
- removed the F5 at (2.48, 1.15)
- removed the F5 at (211.8, 102.9)
- added F5: Fuse_Small, Fuse:Fuse_0805_2012Metric, B.Cu at (211.8, 102.8)
- moved U32 0.11 mm to (232.3, 114.5)
Routing:
- net +5V: track 368.5 -> 369.1 mm

Commit message: Fixed corners
Parts:
- moved U32 0.26 mm to (232.0, 114.5)
Routing:
- removed copper zone on B.Cu, net GND
Changed lines of the file:
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@@
 	(footprint "Frontbox:MODULE_STLINK-V3MODS"
 		(layer "B.Cu")
-		(at 232.256 114.47003 90)
+		(at 232 114.45 90)
 		(property "Reference" "U32"
-			(at -5.075 2.425 270)
+			(at -0.10497 -3.306 -90)
 			(layer "B.SilkS")
 			(effects
@@
 		)
 		(property "Value" "STLINK-V3MODS"
-			(at 4.2 -31.115 270)
+			(at 4.2 -31.115 -90)
 			(layer "B.Fab")
 			(effects
@@
 		)
 	)
-	(gr_line
-		(start 136.407 130.2215)
-		(end 136.407 70.2215)
+	(gr_arc
+		(start 233.407 130.2215)
+		(mid 231.942534 133.757034)
+		(end 228.407 135.2215)
 		(stroke
-			(width 0.4)
+			(width 0.1)
 			(type default)
 		)
@@
 	)
 	(gr_arc
-		(start 141.407 135.2215)
-		(mid 137.871466 133.757034)
-		(end 136.407 130.2215)
+		(start 228.407 65.225)
+		(mid 231.942534 66.689466)
+		(end 233.407 70.225)
 		(stroke
-			(width 0.4)
+			(width 0.1)
 			(type default)
 		)
 		(layer "Edge.Cuts")
 	)
-	(gr_arc
-		(start 136.407 70.2215)
-		(mid 137.871466 66.685966)
-		(end 141.407 65.2215)
+	(gr_line
+		(start 228.407 135.2215)
+		(end 141.41 135.2215)
 		(stroke
-			(width 0.4)
+			(width 0.1)
 			(type default)
 		)
@@
 	)
 	(gr_line
-		(start 141.407 135.2215)
-		(end 228.407 135.2215)
+		(start 233.407 70.225)
+		(end 233.407 130.2215)
 		(stroke
-			(width 0.4)
+			(width 0.1)
 			(type default)
 		)
@@
 	)
 	(gr_arc
-		(start 228.407 65.2215)
-		(mid 231.942534 66.685966)
-		(end 233.407 70.2215)
+		(start 136.41 70.225)
+		(mid 137.874466 66.689466)
+		(end 141.41 65.225)
 		(stroke
-			(width 0.4)
+			(width 0.1)
 			(type default)
 		)
 		(layer "Edge.Cuts")
 	)
-	(gr_line
-		(start 233.407 130.2215)
-		(end 233.407 70.2215)
+	(gr_arc
+		(start 141.41 135.2215)
+		(mid 137.874466 133.757034)
+		(end 136.41 130.2215)
 		(stroke
-			(width 0.4)
+			(width 0.1)
 			(type default)
 		)
 		(layer "Edge.Cuts")
 	)
-	(gr_arc
-		(start 233.407 130.2215)
-		(mid 231.942534 133.757034)
-		(end 228.407 135.2215)
+	(gr_line
+		(start 141.41 65.225)
+		(end 228.407 65.225)
 		(stroke
-			(width 0.4)
+			(width 0.1)
 			(type default)
 		)
@@
 	)
 	(gr_line
-		(start 228.407 65.2215)
-		(end 141.407 65.2215)
+		(start 136.41 130.2215)
+		(end 136.41 70.225)
 		(stroke
-			(width 0.4)
+			(width 0.1)
 			(type default)
 		)
@@
 	)
 	(segment
+		(start 218.284 110.5085)
+		(end 218.284 107.51944)
+		(width 0.6)
+		(layer "B.Cu")
+		(net 2)
+	)
+	(segment
 		(start 218.542 111.3665)
 		(end 218.132 111.7765)
@@
 	)
 	(segment
-		(start 218.542 110.7665)
-		(end 218.542 107.26144)
-		(width 0.6)
+		(start 204.46 98.25)
+		(end 204.4 98.19)
+		(width 0.2)
 		(layer "B.Cu")
 		(net 2)
 	)
 	(segment
-		(start 204.46 98.25)
-		(end 204.4 98.19)
-		(width 0.2)
+		(start 218.542 110.7665)
+		(end 218.284 110.5085)
+		(width 0.6)
 		(layer "B.Cu")
 		(net 2)
@@
 	)
 	(segment
-		(start 207.112 120.75154)
-		(end 207.112 121.9015)
+		(start 203.707 119.9015)
+		(end 206.1265 119.9015)
 		(width 0.2)
 		(layer "B.Cu")
@@
 	)
 	(segment
-		(start 203.707 119.9015)
-		(end 206.26196 119.9015)
+		(start 207.112 120.887)
+		(end 207.112 121.9015)
 		(width 0.2)
 		(layer "B.Cu")
@@
 	)
 	(segment
-		(start 206.26196 119.9015)
-		(end 207.112 120.75154)
+		(start 206.1265 119.9015)
+		(end 207.112 120.887)
 		(width 0.2)
 		(layer "B.Cu")
@@
 	)
 	(segment
-		(start 209.652 105.523)
-		(end 209.652 107.26144)
+		(start 209.4 105.775)
+		(end 209.4 107.00944)
 		(width 0.6)
 		(layer "B.Cu")
@@
 	(segment
 		(start 210.8625 104.3125)
-		(end 209.652 105.523)
+		(end 209.4 105.775)
 		(width 0.6)
 		(layer "B.Cu")
@@
 			)
 		)
-	)
-	(zone
-		(net 2)
-		(net_name "GND")
-		(layer "B.Cu")
-		(hatch edge 0.5)
-		(connect_pads
-			(clearance 0.1)
-		)
-		(min_thickness 0.25)
-		(filled_areas_thickness no)
-		(fill yes
-			(thermal_gap 0.5)
-			(thermal_bridge_width 0.5)
-		)
-		(polygon
-			(pts
-				(xy 136.432 65.2515) (xy 136.432 135.2515) (xy 233.432 135.2515) (xy 233.432 65.8515) (xy 232.832 65.2515)
-			)
-		)
